File: main-board/IMU.sch (KiCad schematic (older format))
At the start: 0 parts

Commit message: Update IMU.sch
Parts:
- added J?: Conn_01x06, symbol Connector_Generic:Conn_01x06
Connections:
- net 3.3V: now also J?.1 (Pin_1)
- net GND: now also J?.3 (Pin_3)
- net SCL: now also J?.5 (Pin_5)
- net SDA: now also J?.4 (Pin_4)
- no-connect marks 0 -> 2
Changed lines of the file:
@@
 Comment4 ""
 $EndDescr
-Text HLabel 2300 2150 0    50   Input ~ 0
+Text HLabel 2400 2150 0    50   Input ~ 0
 SDA
-Text HLabel 2300 2250 0    50   Input ~ 0
+Text HLabel 2400 2250 0    50   Input ~ 0
 SCL
-Text HLabel 2300 1850 0    50   Input ~ 0
+Text HLabel 2400 1850 0    50   Input ~ 0
 3.3V
-Text HLabel 2300 1950 0    50   Input ~ 0
+Text HLabel 2400 2050 0    50   Input ~ 0
 GND
 Text Notes 2200 1450 0    50   ~ 0
 BNO055 IMU\nBreakout board so that the board can be mounted close to center of mass
+$Comp
+L Connector_Generic:Conn_01x06 J?
+U 1 1 60BF9762
+P 3050 2050
+F 0 "J?" H 3130 2042 50  0000 L CNN
+F 1 "Conn_01x06" H 3130 1951 50  0000 L CNN
+F 2 "" H 3050 2050 50  0001 C CNN
+F 3 "~" H 3050 2050 50  0001 C CNN
+	1    3050 2050
+	1    0    0    -1
+$EndComp
+Wire Wire Line
+	2850 1850 2400 1850
+Wire Wire Line
+	2850 2050 2400 2050
+Wire Wire Line
+	2850 2150 2400 2150
+Wire Wire Line
+	2850 2250 2400 2250
+NoConn ~ 2850 1950
+NoConn ~ 2850 2350
 $EndSCHEMATC
