File: main-board/main-board.sch (KiCad schematic (older format))
At the start: 0 parts

Commit message: Got rid of hierarchical sheets
Parts:
- added AE?: Antenna, symbol Device:Antenna
- added BT?: Battery, symbol Device:Battery
- added C?: C_Small, symbol Device:C_Small
- added D?: LED, symbol Device:LED
- added J?: NVIDIA_Jetson_NX_Dev_40pin_Connector, symbol Prototype_Library:NVIDIA_Jetson_NX_Dev_40pin_Connector
- added J?: NVIDIA_Jetson_NX_Dev_Button_Conn, symbol Prototype_Library:NVIDIA_Jetson_NX_Dev_Button_Conn
- added J?: QWIIC_Generic_Conn, symbol ASTRA_Library:QWIIC_Generic_Conn
- added J?: Conn_01x03, symbol Connector_Generic:Conn_01x03
- added J? (x6): FSESC_6.6_COMM, symbol ASTRA_Library:FSESC_6.6_COMM
- added J?: Conn_01x02, symbol Connector_Generic:Conn_01x02
- added M? (x3): Fan_3pin, symbol Motor:Fan_3pin
- added Q? (x6): Q_NMOS_DGS, symbol Device:Q_NMOS_DGS
- added R? (x5): 10k, symbol Device:R_Small
- added R?: 1k, symbol Device:R
- added SW?: SW_SPDT, symbol Switch:SW_SPDT
- added U?: Teensy_4.1, symbol ASTRA_Library:Teensy_4.1
- added U?: RFM95W_Adafruit_Breakout, symbol Prototype_Library:RFM95W_Adafruit_Breakout
- added U? (x5): MCP9700T-HTT, Package_TO_SOT_SMD:SOT-23, symbol Sensor_Temperature:MCP9700T-HTT
- added U?: Sparkfun_OpenLog, symbol Prototype_Library:Sparkfun_OpenLog
- added U?: Adafruit_GPS_V3, symbol ASTRA_Library:Adafruit_GPS_V3
Connections:
- net ADC1: now also U?.16 (P24), U?.2 (Vout)
- net ADC2: now also U?.17 (P25), U?.2 (Vout)
- net ADC3: now also U?.18 (P26), U?.2 (Vout)
- net ADC4: now also U?.19 (P27), U?.2 (Vout)
- net ADC5: now also U?.2 (Vout), U?.33 (P41)
- new net: D?.1 (K), J?.1 (PC_LED-)
- new net: J?.12 (SLEEP/WAKE), Q?.1 (D)
- new net: D?.2 (A), J?.2 (PC_LED+)
- new net: J?.8 (SYS_RESET), Q?.1 (D)
- new net: AE?.1 (A), U?.10 (ANT)
- new net: BT?.1 (+), SW?.1 (A)
- new net: M?.3 (-), Q?.1 (D) (x3)
- new net: J?.3 (Pin_3), Q?.1 (D), R?.2
- new net +12V: J?.1 (Pin_1), M?.2 (+), M?.2 (+), M?.2 (+)
- new net +3V3: J?.2 (3.3V), J?.2 (3.3V), J?.2 (3.3V), J?.2 (3.3V), J?.2 (3.3V), J?.2 (3.3V), Q?.2 (G), U?.1 (Vdd), U?.1 (Vdd), U?.1 (Vdd), U?.1 (Vdd), U?.1 (Vdd)
- new net +5V: C?.1, J?.1 (5V), J?.1 (5V), J?.1 (5V), J?.1 (5V), J?.1 (5V), J?.1 (5V), J?.1 (Pin_1), R?.1
- new net +BATT: SW?.2 (B)
- new net ARGB_Data: Q?.3 (S)
- new net Fan1_Control: Q?.2 (G), R?.1
- new net Fan2_Control: Q?.2 (G), R?.1
- new net Fan3_Control: Q?.2 (G), R?.1
- new net GND: BT?.2 (-), C?.2, J?.11 (GND), J?.2 (Pin_2), J?.2 (Pin_2), J?.3 (GND), J?.3 (GND), J?.3 (GND), J?.3 (GND), J?.3 (GND), J?.3 (GND), J?.7 (GND), J?.9 (GND), Q?.3 (S), Q?.3 (S), Q?.3 (S), Q?.3 (S), Q?.3 (S), R?.2, R?.2, R?.2, R?.2, R?.2, U?.3 (GND), U?.3 (GND), U?.3 (GND), U?.3 (GND), U?.3 (GND)
- new net JETSON_RESET: Q?.2 (G), R?.1
- new net JETSON_SLEEP: Q?.2 (G), R?.1
- new net M1_RX: J?.5 (RX)
- new net M1_TX: J?.6 (TX)
- new net M2_RX: J?.5 (RX)
- new net M2_TX: J?.6 (TX)
- new net M3_RX: J?.5 (RX)
- new net M3_TX: J?.6 (TX)
- new net M4_RX: J?.5 (RX)
- new net M4_TX: J?.6 (TX)
- new net M5_RX: J?.5 (RX)
- new net M5_TX: J?.6 (TX)
- new net M6_RX: J?.5 (RX)
- new net M6_TX: J?.6 (TX)
- no-connect marks 0 -> 22
Other:
- note added: "ARGB Control"
- note added: "Backup Comms"
- note added: "Battery and Switch"
- note added: "Cooling Fans"
- note added: "GPS"
- note added: "IMU"
- note added: "Jetson Power Supply"
- note added: "Motor Driver Connectors"
- note added: "OpenLog"
- note added: "Power Monitor"
- note added: "Power Supply"
- note added: "Temperature Sensors"

Commit message: Teensy Connections
Added the majority of the teensy connections from the excel sheet (minus the coms). Added a few power connections
Connections:
- net +3V3: now also J?.2 (3.3V), U?.1 (Vin)
- net +5V: now also U?.3 (VCC), U?.48 (Vin)
- net ADC1: now also U?.40 (P18); no longer U?.16 (P24)
- net ADC2: now also U?.41 (P19); no longer U?.17 (P25)
- net ARGB_Data: now also U?.4 (P2)
- net Fan1_Control: now also U?.22 (P30)
- net Fan2_Control: now also U?.23 (P31)
- net Fan3_Control: now also U?.24 (P32)
- net GND: now also J?.1 (GND), U?.1 (GND), U?.2 (GND), U?.2 (GND), U?.34 (GND), U?.47 (GND), U?.7 (GND)
- net JETSON_RESET: now also U?.8 (P6)
- net JETSON_SLEEP: now also U?.7 (P5)
- net M1_RX: now also U?.2 (P0)
- net M1_TX: now also U?.3 (P1)
- net M2_RX: now also U?.9 (P7)
- net M2_TX: now also U?.10 (P8)
- net M3_RX: now also U?.37 (P15)
- net M3_TX: now also U?.36 (P14)
- net M4_RX: now also U?.43 (P21)
- net M4_TX: now also U?.42 (P20)
- net M5_RX: now also U?.20 (P28)
- net M5_TX: now also U?.21 (P29)
- net M6_RX: now also U?.26 (P34)
- net M6_TX: now also U?.27 (P35)
- net ADC_3.3V: now reaches U?.30 (P38)
- net ADC_5V: now reaches U?.31 (P39)
- net ADC_BATT: now reaches U?.32 (P40)
- net OPENLOG_RX: now reaches U?.38 (P16)
- net OPENLOG_RX: now also U?.5 (RXI)
- net OPENLOG_TX: now reaches U?.39 (P17)
- net OPENLOG_TX: now also U?.4 (TXO)
- net GPS_TX: now reaches U?.5 (TX)
- net GPS_TX: now also U?.16 (P24)
- net GPS_RX: now reaches U?.6 (RX)
- net GPS_RX: now also U?.17 (P25)
Changed lines of the file:
@@
 EESchema Schematic File Version 4
+LIBS:main-board-cache
 EELAYER 30 0
 EELAYER END
@@
 NoConn ~ 3750 1850
 Wire Wire Line
-	3150 2050 4300 2050
-Wire Wire Line
 	3750 1650 4300 1650
 Text Notes 5450 1150 0    50   ~ 0
@@
 Text Notes 10600 1150 0    50   ~ 0
 Temperature Sensors
-Text Label 6600 6300 2    50   ~ 0
+Text Label 7500 5600 0    50   ~ 0
 ADC1
-Text Label 6600 6400 2    50   ~ 0
+Text Label 7500 5500 0    50   ~ 0
 ADC2
 Text Label 6600 6500 2    50   ~ 0
@@
 	8300 9950 8100 9950
 Connection ~ 8750 10150
+Wire Wire Line
+	3150 2050 4300 2050
+Text Label 6600 4900 2    50   ~ 0
+M1_RX
+Text Label 6600 5000 2    50   ~ 0
+M1_TX
+Text Label 6600 5600 2    50   ~ 0
+M2_RX
+Text Label 6600 5700 2    50   ~ 0
+M2_TX
+Text Label 7500 6000 0    50   ~ 0
+M3_TX
+Text Label 7500 5900 0    50   ~ 0
+M3_RX
+Text Label 6600 6700 2    50   ~ 0
+M5_RX
+Text Label 6600 6800 2    50   ~ 0
+M5_TX
+Text Label 7500 5400 0    50   ~ 0
+M4_TX
+Text Label 7500 5300 0    50   ~ 0
+M4_RX
+Text Label 7500 7000 0    50   ~ 0
+M6_RX
+Text Label 7500 6900 0    50   ~ 0
+M6_TX
+Text Label 6600 5100 2    50   ~ 0
+ARGB_Data
+Text Label 6600 5400 2    50   ~ 0
+JETSON_SLEEP
+Text Label 6600 5500 2    50   ~ 0
+JETSON_RESET
+Text Label 6600 6900 2    50   ~ 0
+Fan1_Control
+Text Label 6600 7000 2    50   ~ 0
+Fan2_Control
+Text Label 6600 7100 2    50   ~ 0
+Fan3_Control
+Text Label 7500 6600 0    50   ~ 0
+ADC_3.3V
+Text Label 7500 6500 0    50   ~ 0
+ADC_5V
+Text Label 7500 6400 0    50   ~ 0
+ADC_BATT
+Text Label 6700 1950 0    50   ~ 0
+ADC_3.3V
+Text Label 6700 1850 0    50   ~ 0
+ADC_5V
+Text Label 6700 1750 0    50   ~ 0
+ADC_BATT
+Text Label 16100 6550 2    50   ~ 0
+OPENLOG_RX
+Text Label 16100 6450 2    50   ~ 0
+OPENLOG_TX
+Text Label 7500 5800 0    50   ~ 0
+OPENLOG_RX
+Text Label 7500 5700 0    50   ~ 0
+OPENLOG_TX
+Text Label 15700 5000 2    50   ~ 0
+GPS_RX
+Text Label 15700 4900 2    50   ~ 0
+GPS_TX
+$Comp
+L power:GND #PWR?
+U 1 1 61098ECE
+P 6200 4800
+F 0 "#PWR?" H 6200 4550 50  0001 C CNN
+F 1 "GND" H 6205 4627 50  0000 C CNN
+F 2 "" H 6200 4800 50  0001 C CNN
+F 3 "" H 6200 4800 50  0001 C CNN
+	1    6200 4800
+	1    0    0    -1
+$EndComp
+$Comp
+L power:GND #PWR?
+U 1 1 61099B4E
+P 8200 6300
+F 0 "#PWR?" H 8200 6050 50  0001 C CNN
+F 1 "GND" H 8205 6127 50  0000 C CNN
+F 2 "" H 8200 6300 50  0001 C CNN
+F 3 "" H 8200 6300 50  0001 C CNN
+	1    8200 6300
+	1    0    0    -1
+$EndComp
+$Comp
+L power:+5V #PWR?
+U 1 1 6109A946
+P 7950 4750
+F 0 "#PWR?" H 7950 4600 50  0001 C CNN
+F 1 "+5V" H 7965 4923 50  0000 C CNN
+F 2 "" H 7950 4750 50  0001 C CNN
+F 3 "" H 7950 4750 50  0001 C CNN
+	1    7950 4750
+	1    0    0    -1
+$EndComp
+Wire Wire Line
+	7950 4750 7950 4800
+Wire Wire Line
+	7950 4800 7500 4800
+Wire Wire Line
+	6200 4800 6600 4800
+$Comp
+L power:GND #PWR?
+U 1 1 610A9769
+P 13600 5050
+F 0 "#PWR?" H 13600 4800 50  0001 C CNN
+F 1 "GND" H 13605 4877 50  0000 C CNN
+F 2 "" H 13600 5050 50  0001 C CNN
+F 3 "" H 13600 5050 50  0001 C CNN
+	1    13600 5050
+	1    0    0    -1
+$EndComp
+$Comp
+L power:GND #PWR?
+U 1 1 610ADE00
+P 15700 5350
+F 0 "#PWR?" H 15700 5100 50  0001 C CNN
+F 1 "GND" H 15705 5177 50  0000 C CNN
+F 2 "" H 15700 5350 50  0001 C CNN
+F 3 "" H 15700 5350 50  0001 C CNN
+	1    15700 5350
+	1    0    0    -1
+$EndComp
+$Comp
+L power:GND #PWR?
+U 1 1 610B2F7E
+P 15800 6050
+F 0 "#PWR?" H 15800 5800 50  0001 C CNN
+F 1 "GND" H 15805 5877 50  0000 C CNN
+F 2 "" H 15800 6050 50  0001 C CNN
+F 3 "" H 15800 6050 50  0001 C CNN
+	1    15800 6050
+	1    0    0    -1
+$EndComp
+$Comp
+L power:GND #PWR?
+U 1 1 610B7464
+P 600 1850
+F 0 "#PWR?" H 600 1600 50  0001 C CNN
+F 1 "GND" H 605 1677 50  0000 C CNN
+F 2 "" H 600 1850 50  0001 C CNN
+F 3 "" H 600 1850 50  0001 C CNN
+	1    600  1850
+	1    0    0    -1
+$EndComp
+$Comp
+L power:+3.3V #PWR?
+U 1 1 610BC0E5
+P 750 1750
+F 0 "#PWR?" H 750 1600 50  0001 C CNN
+F 1 "+3.3V" H 765 1923 50  0000 C CNN
+F 2 "" H 750 1750 50  0001 C CNN
+F 3 "" H 750 1750 50  0001 C CNN
+	1    750  1750
+	1    0    0    -1
+$EndComp
+$Comp
+L power:+3.3V #PWR?
+U 1 1 610BE03A
+P 13100 4850
+F 0 "#PWR?" H 13100 4700 50  0001 C CNN
+F 1 "+3.3V" H 13115 5023 50  0000 C CNN
+F 2 "" H 13100 4850 50  0001 C CNN
+F 3 "" H 13100 4850 50  0001 C CNN
+	1    13100 4850
+	1    0    0    -1
+$EndComp
+$Comp
+L power:+5V #PWR?
+U 1 1 610C39E0
+P 15550 6300
+F 0 "#PWR?" H 15550 6150 50  0001 C CNN
+F 1 "+5V" H 15565 6473 50  0000 C CNN
+F 2 "" H 15550 6300 50  0001 C CNN
+F 3 "" H 15550 6300 50  0001 C CNN
+	1    15550 6300
+	1    0    0    -1
+$EndComp
+Wire Wire Line
+	15950 5100 15700 5100
+Wire Wire Line
+	15700 5100 15700 5350
+Wire Wire Line
+	16100 6250 15900 6250
+Wire Wire Line
+	15900 6250 15900 6050
+Wire Wire Line
+	15900 6050 15800 6050
+Wire Wire Line
+	15550 6300 15550 6350
+Wire Wire Line
+	15550 6350 16100 6350
+Wire Wire Line
+	13100 4850 13750 4850
+Wire Wire Line
+	13600 5050 13600 4950
+Wire Wire Line
+	13600 4950 13750 4950
+Wire Wire Line
+	750  1750 950  1750
+Wire Wire Line
+	950  1850 600  1850
+Wire Wire Line
+	7500 4900 8200 4900
+Wire Wire Line
+	7500 6200 8200 6200
+Wire Wire Line
+	8200 6200 8200 4900
+Wire Wire Line
+	8200 6300 8200 6200
+Connection ~ 8200 6200
+Wire Wire Line
+	15950 4900 15700 4900
+Wire Wire Line
+	15950 5000 15700 5000
+Text Label 6600 6400 2    50   ~ 0
+GPS_RX
+Text Label 6600 6300 2    50   ~ 0
+GPS_TX
 $EndSCHEMATC

Commit message: changed a few thingies
Connections:
- net +3V3: now also U?.3 (VCC), U?.8 (VIN); no longer J?.2 (3.3V), J?.2 (3.3V), J?.2 (3.3V), J?.2 (3.3V), J?.2 (3.3V), J?.2 (3.3V)
- net +5V: no longer J?.1 (5V), J?.1 (5V), J?.1 (5V), J?.1 (5V), J?.1 (5V), J?.1 (5V), U?.3 (VCC)
- net NX_SDA: now reaches J?.3 (I2C1_SDA)
- net NX_SDA: now also J?.3 (SDA)
- net NX_SCL: now reaches J?.5 (I2C1_SCL)
- net NX_SCL: now also J?.4 (SCL)
- net COMMS_CS: now reaches U?.12 (P10)
- net COMMS_CS: now also U?.8 (CS)
- net MOSI: now reaches U?.13 (P11)
- net MOSI: now also U?.7 (MOSI)
- net MISO: now reaches U?.14 (P12)
- net MISO: now also U?.6 (MISO)
- net SCK: now reaches U?.35 (P13)
- net SCK: now also U?.5 (SCK)
- net COMMS_RST: now reaches U?.5 (P3)
- net COMMS_RST: now also U?.9 (RST)
- net COMMS_G0: now reaches U?.6 (P4)
- net COMMS_G0: now also U?.4 (G0)
- no-connect marks 22 -> 23

Commit message: small tweaks
Connections:
- net Fan1_Control: now also U?.25 (P33); no longer U?.22 (P30)
- net Fan2_Control: now also U?.28 (P36); no longer U?.23 (P31)
- net Fan3_Control: now also U?.29 (P37); no longer U?.24 (P32)
- net GND: now also J?.14 (GND), J?.20 (GND), J?.25 (GND), J?.30 (GND), J?.34 (GND), J?.39 (GND), J?.6 (GND), J?.9 (GND)
Changed lines of the file:
@@
 Text Label 6600 5500 2    50   ~ 0
 JETSON_RESET
-Text Label 6600 6900 2    50   ~ 0
+Text Label 7500 7100 0    50   ~ 0
 Fan1_Control
-Text Label 6600 7000 2    50   ~ 0
+Text Label 7500 6800 0    50   ~ 0
 Fan2_Control
-Text Label 6600 7100 2    50   ~ 0
+Text Label 7500 6700 0    50   ~ 0
 Fan3_Control
 Text Label 7500 6600 0    50   ~ 0
@@
 Wire Wire Line
 	9400 5350 9300 5350
+$Comp
+L power:GND #PWR?
+U 1 1 6112AD47
+P 9100 7200
+F 0 "#PWR?" H 9100 6950 50  0001 C CNN
+F 1 "GND" H 9105 7027 50  0000 C CNN
+F 2 "" H 9100 7200 50  0001 C CNN
+F 3 "" H 9100 7200 50  0001 C CNN
+	1    9100 7200
+	1    0    0    -1
+$EndComp
+Wire Wire Line
+	9100 7200 9100 7050
+Wire Wire Line
+	9100 5550 9400 5550
+Wire Wire Line
+	9400 6350 9100 6350
+Connection ~ 9100 6350
+Wire Wire Line
+	9100 6350 9100 5550
+Wire Wire Line
+	9400 7050 9100 7050
+Connection ~ 9100 7050
+Wire Wire Line
+	9100 7050 9100 6350
+$Comp
+L power:GND #PWR?
+U 1 1 6113B29F
+P 10900 7200
+F 0 "#PWR?" H 10900 6950 50  0001 C CNN
+F 1 "GND" H 10905 7027 50  0000 C CNN
+F 2 "" H 10900 7200 50  0001 C CNN
+F 3 "" H 10900 7200 50  0001 C CNN
+	1    10900 7200
+	1    0    0    -1
+$EndComp
+Wire Wire Line
+	10600 5350 10900 5350
+Wire Wire Line
+	10900 5350 10900 5750
+Wire Wire Line
+	10600 6750 10900 6750
+Connection ~ 10900 6750
+Wire Wire Line
+	10900 6750 10900 7200
+Wire Wire Line
+	10600 6550 10900 6550
+Connection ~ 10900 6550
+Wire Wire Line
+	10900 6550 10900 6750
+Wire Wire Line
+	10600 6050 10900 6050
+Connection ~ 10900 6050
+Wire Wire Line
+	10900 6050 10900 6550
+Wire Wire Line
+	10600 5750 10900 5750
+Connection ~ 10900 5750
+Wire Wire Line
+	10900 5750 10900 6050
 $EndSCHEMATC

Commit message: started work on power supplies
Parts:
- added U?: Pololu_4095, symbol ASTRA_Library:Pololu_4095
Connections:
- net +12V: now also U?.1 (VOUT), U?.12 (VOUT)
- net +BATT: now also U?.4 (VIN), U?.9 (VIN)
- net GND: now also U?.10 (GND), U?.11 (GND), U?.2 (GND), U?.3 (GND)
- no-connect marks 23 -> 27
Other:
- note added: "12v"
- note added: "24v"
- note added: "3.3v"
- note added: "5v"
- note added: "Power Supplies"
- note removed: "Power Supply"
Changed lines of the file:
@@
 	3750 1650 4300 1650
 Text Notes 5450 1150 0    50   ~ 0
-Power Supply
+Power Supplies
 Text Notes 3450 1150 0    50   ~ 0
 Battery and Switch
@@
 Text Label 7500 6400 0    50   ~ 0
 ADC_BATT
-Text Label 7250 2150 0    50   ~ 0
+Text Label 7500 2100 0    50   ~ 0
 ADC_3.3V
-Text Label 7250 2050 0    50   ~ 0
+Text Label 7500 2000 0    50   ~ 0
 ADC_5V
-Text Label 7250 1950 0    50   ~ 0
+Text Label 7500 1900 0    50   ~ 0
 ADC_BATT
 Text Label 16100 6550 2    50   ~ 0
@@
 Wire Wire Line
 	10900 5750 10900 6050
+$Comp
+L ASTRA_Library:Pololu_4095 U?
+U 1 1 611619B4
+P 5700 2050
+F 0 "U?" H 5700 2565 50  0000 C CNN
+F 1 "Pololu_4095" H 5700 2474 50  0000 C CNN
+F 2 "" H 5700 2050 50  0001 C CNN
+F 3 "" H 5700 2050 50  0001 C CNN
+	1    5700 2050
+	1    0    0    -1
+$EndComp
+$Comp
+L power:+12V #PWR?
+U 1 1 6116292A
+P 5150 1800
+F 0 "#PWR?" H 5150 1650 50  0001 C CNN
+F 1 "+12V" H 5165 1973 50  0000 C CNN
+F 2 "" H 5150 1800 50  0001 C CNN
+F 3 "" H 5150 1800 50  0001 C CNN
+	1    5150 1800
+	1    0    0    -1
+$EndComp
+Wire Wire Line
+	5150 1800 5350 1800
+$Comp
+L power:+12V #PWR?
+U 1 1 61169CED
+P 6300 1800
+F 0 "#PWR?" H 6300 1650 50  0001 C CNN
+F 1 "+12V" H 6315 1973 50  0000 C CNN
+F 2 "" H 6300 1800 50  0001 C CNN
+F 3 "" H 6300 1800 50  0001 C CNN
+	1    6300 1800
+	1    0    0    -1
+$EndComp
+Wire Wire Line
+	6300 1800 6050 1800
+$Comp
+L power:GND #PWR?
+U 1 1 6117098E
+P 5050 1900
+F 0 "#PWR?" H 5050 1650 50  0001 C CNN
+F 1 "GND" H 5055 1727 50  0000 C CNN
+F 2 "" H 5050 1900 50  0001 C CNN
+F 3 "" H 5050 1900 50  0001 C CNN
+	1    5050 1900
+	1    0    0    -1
+$EndComp
+Wire Wire Line
+	5350 1900 5150 1900
+Wire Wire Line
+	5150 1900 5150 2000
+Wire Wire Line
+	5350 2000 5150 2000
+$Comp
+L power:GND #PWR?
+U 1 1 6117E9FE
+P 6400 1900
+F 0 "#PWR?" H 6400 1650 50  0001 C CNN
+F 1 "GND" H 6405 1727 50  0000 C CNN
+F 2 "" H 6400 1900 50  0001 C CNN
+F 3 "" H 6400 1900 50  0001 C CNN
+	1    6400 1900
+	1    0    0    -1
+$EndComp
+Wire Wire Line
+	6300 2000 6300 1900
+Wire Wire Line
+	6300 1900 6050 1900
+Wire Wire Line
+	6050 2000 6300 2000
+$Comp
+L power:+BATT #PWR?
+U 1 1 6118D321
+P 4850 2100
+F 0 "#PWR?" H 4850 1950 50  0001 C CNN
+F 1 "+BATT" H 4865 2273 50  0000 C CNN
+F 2 "" H 4850 2100 50  0001 C CNN
+F 3 "" H 4850 2100 50  0001 C CNN
+	1    4850 2100
+	1    0    0    -1
+$EndComp
+$Comp
+L power:+BATT #PWR?
+U 1 1 6119629D
+P 6600 2100
+F 0 "#PWR?" H 6600 1950 50  0001 C CNN
+F 1 "+BATT" H 6615 2273 50  0000 C CNN
+F 2 "" H 6600 2100 50  0001 C CNN
+F 3 "" H 6600 2100 50  0001 C CNN
+	1    6600 2100
+	1    0    0    -1
+$EndComp
+Wire Wire Line
+	5150 1900 5050 1900
+Connection ~ 5150 1900
+Wire Wire Line
+	4850 2100 5350 2100
+Wire Wire Line
+	6400 1900 6300 1900
+Connection ~ 6300 1900
+Wire Wire Line
+	6050 2100 6600 2100
+NoConn ~ 5350 2200
+NoConn ~ 6050 2200
+NoConn ~ 5350 2300
+NoConn ~ 6050 2300
+Text Notes 5650 1400 0    50   ~ 0
+12v
+Text Notes 5600 2750 0    50   ~ 0
+24v
+Text Notes 5600 3150 0    50   ~ 0
+5v
+Text Notes 5600 3550 0    50   ~ 0
+3.3v
 $EndSCHEMATC

Commit message: More work on power supply stuff
Parts:
- removed SW?: SW_SPDT, symbol Switch:SW_SPDT
- removed U?: Pololu_4095, symbol ASTRA_Library:Pololu_4095
- added C? (x2): 33u, symbol Device:CP_Small
- added D? (x6): D_Schottky_Small, symbol Device:D_Schottky_Small
- added J?: Conn_01x02, symbol Connector_Generic:Conn_01x02
- added Q? (x2): Q_NMOS_DGS, symbol Device:Q_NMOS_DGS
- added R? (x2): 100k, symbol Device:R_Small
- added R?: 1.82k, symbol Device:R_Small
- added R?: 8.57k, symbol Device:R_Small
- added R? (x3): 10k, symbol Device:R_Small
- added R? (x3): 80.6k, symbol Device:R_Small
- added U? (x2): TDK_I3A4W008A033V, symbol ASTRA_Library:TDK_I3A4W008A033V
Connections:
- net ADC_3.3V is gone; now on net ADC_5V: U?.30 (P38)
- net +12V: now also J?.1 (Pin_1), R?.1, R?.1, U?.7 (SENSE+), U?.8 (VOUT+)
- net +3V3: now also U?.46 (3.3V), D?.1 (K), D?.1 (K), D?.1 (K)
- net +5V: now also R?.1, R?.1, U?.7 (SENSE+), U?.8 (VOUT+)
- net +BATT: now also BT?.1 (+), C?.1, C?.1, R?.1, U?.1 (VIN+), U?.1 (VIN+)
- net ADC_5V: now also D?.1 (K), D?.2 (A), R?.1, R?.2; no longer U?.31 (P39)
- net ADC_BATT: now also D?.1 (K), D?.2 (A), R?.1, R?.2
- net GND: now also C?.2, C?.2, D?.2 (A), D?.2 (A), D?.2 (A), J?.2 (Pin_2), Q?.3 (S), Q?.3 (S), R?.2, R?.2, R?.2, R?.2, R?.2, U?.3 (VIN-), U?.3 (VIN-), U?.4 (VOUT-), U?.4 (VOUT-)
- net 12V_Disable: now reaches U?.22 (P30)
- net 12V_Disable: now also Q?.2 (G), R?.1
- net 5V_Disable: now reaches U?.23 (P31)
- net 5V_Disable: now also Q?.2 (G), R?.1
- new net: Q?.1 (D), U?.2 (ON/OFF) (x2)
- new net: R?.2, U?.6 (TRIM) (x2)
- new net ADC_12V: D?.1 (K), D?.2 (A), R?.1, R?.2, U?.31 (P39)
- no-connect marks 27 -> 24
Other:
- note added: "Removed switch since it'll need to be off-board"
- note added: "This part may not reliably reset\nIf this is the case, don't populate this MOSFET"
- note added: "off-board PSD-30B-24"
- note removed: "3.3v"
- moved on the sheet: AE?, BT?, U?

Commit message: Lots of small changes
Parts:
- removed C?: C_Small, symbol Device:C_Small
- removed Q?: Q_NMOS_DGS, symbol Device:Q_NMOS_DGS
- removed R?: 1k, symbol Device:R
- added C?: 100n, symbol Device:C_Small
- added C?: 1000u, symbol Device:CP_Small
- added D? (x3): D_Schottky_Small, symbol Device:D_Schottky_Small
- added J5: Conn_01x02, symbol Connector_Generic:Conn_01x02
- added U?: SN74AHCT125D, symbol ASTRA_Library:SN74AHCT125D
- gave numbers to parts that had none: 59
Connections:
- net +12V: now also D?.1 (K), D?.1 (K), D?.1 (K), J5.1 (Pin_1)
- net +5V: now also C?.1, C?.1, U?.14 (VCC)
- net ARGB_Data: now also U?.2 (1A)
- net GND: now also C?.2, C?.2, J5.2 (Pin_2), U?.1 (1~OE), U?.10 (3~OE), U?.11 (4Y), U?.12 (4A), U?.13 (4~OE), U?.4 (2~OE), U?.5 (2A), U?.6 (2Y), U?.7 (GND), U?.8 (3Y), U?.9 (3A)
- net at M1.3 (-), Q6.1 (D): now also D?.2 (A)
- net at M2.3 (-), Q7.1 (D): now also D?.2 (A)
- net at M3.3 (-), Q8.1 (D): now also D?.2 (A)
- net at J7.3 (Pin_3): now also U?.3 (1Y)
Other:
- note added: "Network Switch Power Supply"
- note added: "PTZ Camera Power Supply"
