File: main-board/main-board.sch (KiCad schematic (older format))
At the start: 66 parts, among them J1 NVIDIA_Jetson_NX_Dev_40pin_Co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, J10 FSESC_6.6_COMM, J11 FSESC_6.6_COMM, J12 FSESC_6.6_COMM, J13 FSESC_6.6_COMM, J2 NVIDIA_Jetson_NX_Dev_Button_C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, J3 Conn_01x02, J4 Conn_01x02, J5 Conn_01x02, J6 QWIIC_Generic_Conn, J7 Conn_01x03, J8 FSESC_6.6_COMM, J9 FSESC_6.6_COMM, M1 Fan_3pin, M2 Fan_3pin, M3 Fan_3pin, Q1 Q_NMOS_DGS, Q2 Q_NMOS_DGS, Q3 Q_NMOS_DGS, Q4 Q_NMOS_DGS, Q6 Q_NMOS_DGS, Q7 Q_NMOS_DGS, Q8 Q_NMOS_DGS, U1 RFM95W_Adafruit_Breakout, U10 Adafruit_GPS_V3, U11 Sparkfun_OpenLog, U2 TDK_I3A4W008A033V, U3 TDK_I3A4W008A033V, U4 Teensy_4.1, U5 MCP9700T-HTT, U6 MCP9700T-HTT, U7 MCP9700T-HTT, U8 MCP9700T-HTT, U9 MCP9700T-HTT

Commit message: started sourcing components
Parts:
- removed AE1: Antenna, symbol Device:Antenna
- C1, C2: Digikey Part Num (none) -> 493-2137-1-ND
- C3: renamed from C?; Digikey Part Num (none) -> 493-10756-1-ND
- C4: renamed from C?; Digikey Part Num (none) -> 1276-1941-1-ND
- D1, D2, D3, D4, D5, D6: Digikey Part Num (none) -> 1514-CMDD6001TRPBFREECT-ND
- D10, D8, D9: renamed from D?; Digikey Part Num (none) -> 1655-1927-1-ND
- D7: Digikey Part Num (none) -> 732-4980-1-ND
- gave numbers to parts that had none: 1
Connections:
- no-connect marks 24 -> 25
Other:
- note added: "ANT connection off-board"
Changed lines of the file:
@@
 F 2 "" H 9300 8650 50  0001 C CNN
 F 3 "~" H 9300 8650 50  0001 C CNN
+F 4 "732-4980-1-ND" H 9300 8650 50  0001 C CNN "Digikey Part Num"
 	1    9300 8650
 	1    0    0    -1
@@
 	1    0    0    -1
 $EndComp
-$Comp
-L Device:Antenna AE?
-U 1 1 60FD941A
-P 2350 2350
-AR Path="/60809DA2/60FD941A" Ref="AE?"  Part="1"
-AR Path="/60FD941A" Ref="AE1"  Part="1"
-F 0 "AE1" H 2430 2339 50  0000 L CNN
-F 1 "Antenna" H 2430 2248 50  0000 L CNN
-F 2 "" H 2350 2350 50  0001 C CNN
-F 3 "~" H 2350 2350 50  0001 C CNN
-	1    2350 2350
-	1    0    0    -1
-$EndComp
-Wire Wire Line
-	2350 2550 2100 2550
 $Comp
 L Device:Battery BT?
@@
 F 2 "" V 3750 1960 50  0001 C CNN
 F 3 "~" V 3750 1960 50  0001 C CNN
+F 4 "~" H 3750 1900 50  0001 C CNN "Digikey Part Num"
 	1    3750 1900
 	1    0    0    -1
@@
 F 2 "" H 2300 4800 50  0001 C CNN
 F 3 "~" H 2300 4800 50  0001 C CNN
+F 4 "493-2137-1-ND" H 2300 4800 50  0001 C CNN "Digikey Part Num"
 	1    2300 4800
 	0    1    1    0
@@
 F 2 "" H 2750 6800 50  0001 C CNN
 F 3 "~" H 2750 6800 50  0001 C CNN
+F 4 "493-2137-1-ND" H 2750 6800 50  0001 C CNN "Digikey Part Num"
 	1    2750 6800
 	0    1    1    0
@@
 F 2 "" V 5750 2000 50  0001 C CNN
 F 3 "~" V 5750 2000 50  0001 C CNN
+F 4 "1514-CMDD6001TRPBFREECT-ND" H 5750 2000 50  0001 C CNN "Digikey Part Num"
 	1    5750 2000
 	0    1    1    0
@@
 F 2 "" V 5750 2300 50  0001 C CNN
 F 3 "~" V 5750 2300 50  0001 C CNN
+F 4 "1514-CMDD6001TRPBFREECT-ND" H 5750 2300 50  0001 C CNN "Digikey Part Num"
 	1    5750 2300
 	0    1    1    0
@@
 F 2 "" V 5750 3100 50  0001 C CNN
 F 3 "~" V 5750 3100 50  0001 C CNN
+F 4 "1514-CMDD6001TRPBFREECT-ND" H 5750 3100 50  0001 C CNN "Digikey Part Num"
 	1    5750 3100
 	0    1    1    0
@@
 F 2 "" V 5750 3400 50  0001 C CNN
 F 3 "~" V 5750 3400 50  0001 C CNN
+F 4 "1514-CMDD6001TRPBFREECT-ND" H 5750 3400 50  0001 C CNN "Digikey Part Num"
 	1    5750 3400
 	0    1    1    0
@@
 F 2 "" V 7500 3100 50  0001 C CNN
 F 3 "~" V 7500 3100 50  0001 C CNN
+F 4 "1514-CMDD6001TRPBFREECT-ND" H 7500 3100 50  0001 C CNN "Digikey Part Num"
 	1    7500 3100
 	0    1    1    0
@@
 F 2 "" V 7500 3400 50  0001 C CNN
 F 3 "~" V 7500 3400 50  0001 C CNN
+F 4 "1514-CMDD6001TRPBFREECT-ND" H 7500 3400 50  0001 C CNN "Digikey Part Num"
 	1    7500 3400
 	0    1    1    0
@@
 PTZ Camera Power Supply
 $Comp
-L ASTRA_Library:SN74AHCT125D U?
+L ASTRA_Library:SN74AHCT125D U12
 U 1 1 6140A0D6
 P 17650 3000
-F 0 "U?" H 17650 3565 50  0000 C CNN
+F 0 "U12" H 17650 3565 50  0000 C CNN
 F 1 "SN74AHCT125D" H 17650 3474 50  0000 C CNN
 F 2 "" H 17300 3400 50  0001 C CNN
@@
 $EndComp
 $Comp
-L power:+5V #PWR?
+L power:+5V #PWR068
 U 1 1 6140C53D
 P 18350 2700
-F 0 "#PWR?" H 18350 2550 50  0001 C CNN
+F 0 "#PWR068" H 18350 2550 50  0001 C CNN
 F 1 "+5V" H 18365 2873 50  0000 C CNN
 F 2 "" H 18350 2700 50  0001 C CNN
@@
 	17300 2800 16850 2800
 $Comp
-L power:GND #PWR?
+L power:GND #PWR054
 U 1 1 6146674B
 P 17150 3300
-F 0 "#PWR?" H 17150 3050 50  0001 C CNN
+F 0 "#PWR054" H 17150 3050 50  0001 C CNN
 F 1 "GND" H 17155 3127 50  0000 C CNN
 F 2 "" H 17150 3300 50  0001 C CNN
@@
 	17150 3200 17150 3300
 $Comp
-L power:GND #PWR?
+L power:GND #PWR055
 U 1 1 6149A414
 P 18150 3300
-F 0 "#PWR?" H 18150 3050 50  0001 C CNN
+F 0 "#PWR055" H 18150 3050 50  0001 C CNN
 F 1 "GND" H 18155 3127 50  0000 C CNN
 F 2 "" H 18150 3300 50  0001 C CNN
@@
 P 18350 2800
 AR Path="/607506EB/61532D9F" Ref="C?"  Part="1"
-AR Path="/61532D9F" Ref="C?"  Part="1"
-F 0 "C?" H 18442 2846 50  0000 L CNN
+AR Path="/61532D9F" Ref="C4"  Part="1"
+F 0 "C4" H 18442 2846 50  0000 L CNN
 F 1 "100n" H 18442 2755 50  0000 L CNN
 F 2 "" H 18350 2800 50  0001 C CNN
 F 3 "~" H 18350 2800 50  0001 C CNN
+F 4 "1276-1941-1-ND" H 18350 2800 50  0001 C CNN "Digikey Part Num"
 	1    18350 2800
 	1    0    0    -1
@@
 Connection ~ 18350 2700
 $Comp
-L power:GND #PWR?
+L power:GND #PWR069
 U 1 1 615422B8
 P 18350 2900
-F 0 "#PWR?" H 18350 2650 50  0001 C CNN
+F 0 "#PWR069" H 18350 2650 50  0001 C CNN
 F 1 "GND" H 18355 2727 50  0000 C CNN
 F 2 "" H 18350 2900 50  0001 C CNN
@@
 $EndComp
 $Comp
-L Device:CP_Small C?
+L Device:CP_Small C3
 U 1 1 615516EA
 P 16550 2150
-F 0 "C?" H 16638 2196 50  0000 L CNN
+F 0 "C3" H 16638 2196 50  0000 L CNN
 F 1 "1000u" H 16638 2105 50  0000 L CNN
 F 2 "" H 16550 2150 50  0001 C CNN
 F 3 "~" H 16550 2150 50  0001 C CNN
+F 4 "493-10756-1-ND" H 16550 2150 50  0001 C CNN "Digikey Part Num"
 	1    16550 2150
 	1    0    0    -1
 $EndComp
 $Comp
-L Device:D_Schottky_Small D?
+L Device:D_Schottky_Small D8
 U 1 1 61552B09
 P 20550 9700
-F 0 "D?" V 20504 9770 50  0000 L CNN
+F 0 "D8" V 20504 9770 50  0000 L CNN
 F 1 "D_Schottky_Small" V 20595 9770 50  0000 L CNN
 F 2 "" V 20550 9700 50  0001 C CNN
 F 3 "~" V 20550 9700 50  0001 C CNN
+F 4 "1655-1927-1-ND" H 20550 9700 50  0001 C CNN "Digikey Part Num"
 	1    20550 9700
 	0    1    1    0
@@
 	19900 10000 19900 10100
 $Comp
-L Device:D_Schottky_Small D?
+L Device:D_Schottky_Small D9
 U 1 1 6158E1BB
 P 20550 11600
-F 0 "D?" V 20504 11670 50  0000 L CNN
+F 0 "D9" V 20504 11670 50  0000 L CNN
 F 1 "D_Schottky_Small" V 20595 11670 50  0000 L CNN
 F 2 "" V 20550 11600 50  0001 C CNN
 F 3 "~" V 20550 11600 50  0001 C CNN
+F 4 "1655-1927-1-ND" H 20550 11600 50  0001 C CNN "Digikey Part Num"
 	1    20550 11600
 	0    1    1    0
@@
 	19900 11900 19900 12000
 $Comp
-L Device:D_Schottky_Small D?
+L Device:D_Schottky_Small D10
 U 1 1 6159E9D3
 P 20550 13500
-F 0 "D?" V 20504 13570 50  0000 L CNN
+F 0 "D10" V 20504 13570 50  0000 L CNN
 F 1 "D_Schottky_Small" V 20595 13570 50  0000 L CNN
 F 2 "" V 20550 13500 50  0001 C CNN
 F 3 "~" V 20550 13500 50  0001 C CNN
+F 4 "1655-1927-1-ND" H 20550 13500 50  0001 C CNN "Digikey Part Num"
 	1    20550 13500
 	0    1    1    0
@@
 Wire Wire Line
 	19900 13800 19900 13900
+NoConn ~ 2100 2550
+Text Notes 2200 2550 0    50   ~ 0
+ANT connection off-board
 $EndSCHEMATC
