File: main-board/main-board.sch (KiCad schematic (older format))
At the start: 65 parts, among them J1 NVIDIA_Jetson_NX_Dev_40pin_Co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, J10 FSESC_6.6_COMM, J11 FSESC_6.6_COMM, J12 FSESC_6.6_COMM, J13 FSESC_6.6_COMM, J2 NVIDIA_Jetson_NX_Dev_Button_C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, J3 Conn_01x02, J4 Conn_01x02, J5 Conn_01x02, J6 QWIIC_Generic_Conn, J7 Conn_01x03, J8 FSESC_6.6_COMM, J9 FSESC_6.6_COMM, M1 Fan_3pin, M2 Fan_3pin, M3 Fan_3pin, Q1 Q_NMOS_DGS, Q2 Q_NMOS_DGS, Q3 Q_NMOS_DGS, Q4 Q_NMOS_DGS, Q6 Q_NMOS_DGS, Q7 Q_NMOS_DGS, Q8 Q_NMOS_DGS, U1 RFM95W_Adafruit_Breakout, U10 Adafruit_GPS_V3, U11 Sparkfun_OpenLog, U12 SN74AHCT125D, U2 TDK_I3A4W008A033V, U3 TDK_I3A4W008A033V, U4 Teensy_4.1, U5 MCP9700T-HTT, U6 MCP9700T-HTT, U7 MCP9700T-HTT, U8 MCP9700T-HTT, U9 MCP9700T-HTT

Commit message: Parts selected
Parts:
- J1: Digikey Part Num (none) -> S9175-ND
- J10, J11, J12, J13, J7, J8, J9: Digikey Part Num (none) -> ~ JST PH
- J3, J4, J5: Digikey Part Num (none) -> 455-2247-ND
- J6: Digikey Part Num (none) -> 455-1804-1-ND
- Q1, Q2, Q3, Q4: Digikey Part Num (none) -> SSM3K2615RLFCT-ND
- Q5: renamed from Q6; Digikey Part Num (none) -> SSM3K2615RLFCT-ND
- Q6: renamed from Q7; Digikey Part Num (none) -> SSM3K2615RLFCT-ND
- Q7: renamed from Q8; Digikey Part Num (none) -> SSM3K2615RLFCT-ND
- R1, R2: Digikey Part Num (none) -> 311-100KHRCT-ND
- R10, R11, R12, R6, R8: Digikey Part Num (none) -> 311-10.0KHRCT-ND
- R13: renamed from R14; Digikey Part Num (none) -> 311-10.0KHRCT-ND
- R14: renamed from R15; Digikey Part Num (none) -> 311-10.0KHRCT-ND
- R15: renamed from R16; Digikey Part Num (none) -> 311-10.0KHRCT-ND
- R3: Digikey Part Num (none) -> 311-1.82KHRCT-ND
- R4: value 8.57k -> 8.45k; Digikey Part Num (none) -> 311-8.45KHRCT-ND
- R5, R7, R9: Digikey Part Num (none) -> P20500CT-ND
- U1: Digikey Part Num (none) -> 1528-1667-ND
- U10: Digikey Part Num (none) -> 1528-1153-ND
- U11: Digikey Part Num (none) -> 1568-1368-ND
- U4: Digikey Part Num (none) -> 1568-DEV-16771-ND
- U5, U6, U7, U8, U9: value MCP9700T-HTT -> Analog Temp Sensor; Digikey Part Num (none) -> 296-46127-1-ND

Commit message: Set a lot of footprints
Parts:
- BT1: footprint (none) -> Connector_AMASS:AMASS_XT60-M_1x02_P7.20mm_Vertical
- C1, C2: footprint (none) -> Capacitor_SMD:CP_Elec_8x5.4
- C3: footprint (none) -> Capacitor_THT:CP_Radial_D8.0mm_P3.50mm
- C4: footprint (none) -> Capacitor_SMD:C_0603_1608Metric
- D1, D2, D3, D4, D5, D6: footprint (none) -> Diode_SMD:D_SOD-323_HandSoldering
- D10, D8, D9: footprint (none) -> Diode_SMD:D_SOD-123F
- D7: footprint (none) -> LED_SMD:LED_0603_1608Metric_Pad1.05x0.95mm_HandSolder
- J1: footprint (none) -> Connector_IDC:IDC-Header_2x20_P2.54mm_Vertical
- J10, J11, J12, J13, J8, J9: footprint (none) -> Connector_JST:JST_PH_B8B-PH-K_1x08_P2.00mm_Vertical
- J2: footprint (none) -> Connector_PinHeader_2.54mm:PinHeader_1x12_P2.54mm_Vertical
- J3, J4, J5: footprint (none) -> Connector_JST:JST_XH_B2B-XH-A_1x02_P2.50mm_Vertical
- J6: footprint (none) -> Connector_JST:JST_SH_SM04B-SRSS-TB_1x04-1MP_P1.00mm_Horizontal
- J7: footprint (none) -> Connector_JST:JST_PH_B3B-PH-K_1x03_P2.00mm_Vertical
- M1, M2, M3: footprint (none) -> Connector_Molex:Molex_KK-254_AE-6410-03A_1x03_P2.54mm_Vertical; symbol Motor:Fan_3pin -> ASTRA_Library:Fan_Tacho_Reversed; Digikey Part Num (none) -> WM2701-ND
- Q1, Q2, Q3, Q4, Q5, Q6, Q7: value Q_NMOS_DGS -> Q_NMOS_GSD; footprint (none) -> Package_TO_SOT_SMD:SOT-23; symbol Device:Q_NMOS_DGS -> Device:Q_NMOS_GSD
- R1, R10, R11, R12, R13, R14, R15, R2, R3, R4, R5, R6, R7, R8, R9: footprint (none) -> Resistor_SMD:R_0603_1608Metric
- U12: footprint (none) -> Package_SO:SOIC-14_3.9x8.7mm_P1.27mm

Commit message: started PCB
Parts:
- removed U11: Sparkfun_OpenLog, symbol Prototype_Library:Sparkfun_OpenLog
- U1: footprint (none) -> ASTRA_Footprints:Adafruit_RFM95W
- U10: footprint (none) -> ASTRA_Footprints:Adafruit_GPS_Breakout
- U2, U3: footprint (none) -> ASTRA_Footprints:Power_Supply_32nd_Brick
- U4: footprint (none) -> ASTRA_Footprints:Teensy4.1
Connections:
- net labels removed: OPENLOG_RX, OPENLOG_TX
- wire segments 232 -> 227
Other:
- note removed: "OpenLog"
Changed lines of the file:
@@
 F 0 "U4" H 7050 7365 50  0000 C CNN
 F 1 "Teensy_4.1" H 7050 7274 50  0000 C CNN
-F 2 "" H 7050 5950 50  0001 C CNN
+F 2 "ASTRA_Footprints:Teensy4.1" H 7050 5950 50  0001 C CNN
 F 3 "" H 7050 5950 50  0001 C CNN
 F 4 "1568-DEV-16771-ND" H 7050 5950 50  0001 C CNN "Digikey Part Num"
@@
 F 0 "U1" H 1625 2815 50  0000 C CNN
 F 1 "RFM95W_Adafruit_Breakout" H 1625 2724 50  0000 C CNN
-F 2 "" H 1650 2150 50  0001 C CNN
+F 2 "ASTRA_Footprints:Adafruit_RFM95W" H 1650 2150 50  0001 C CNN
 F 3 "" H 1650 2150 50  0001 C CNN
 F 4 "1528-1667-ND" H 1650 2150 50  0001 C CNN "Digikey Part Num"
@@
 Fan3_Control
 $Comp
-L Prototype_Library:Sparkfun_OpenLog U11
-U 1 1 6100C73E
-P 16350 6400
-F 0 "U11" H 16528 6451 50  0000 L CNN
-F 1 "Sparkfun_OpenLog" H 16528 6360 50  0000 L CNN
-F 2 "" H 16350 6400 50  0001 C CNN
-F 3 "" H 16350 6400 50  0001 C CNN
-F 4 "1568-1368-ND" H 16350 6400 50  0001 C CNN "Digikey Part Num"
-	1    16350 6400
-	1    0    0    -1
-$EndComp
-$Comp
 L ASTRA_Library:Adafruit_GPS_V3 U10
 U 1 1 610109FB
@@
 F 0 "U10" H 16528 4746 50  0000 L CNN
 F 1 "Adafruit_GPS_V3" H 16528 4655 50  0000 L CNN
-F 2 "" H 16250 4800 50  0001 C CNN
+F 2 "ASTRA_Footprints:Adafruit_GPS_Breakout" H 16250 4800 50  0001 C CNN
 F 3 "" H 16250 4800 50  0001 C CNN
 F 4 "1528-1153-ND" H 16250 4800 50  0001 C CNN "Digikey Part Num"
@@
 Text Notes 13900 4200 0    50   ~ 0
 IMU
-Text Notes 16200 5850 0    50   ~ 0
-OpenLog
 Text Notes 19750 8800 0    50   ~ 0
 Cooling Fans
@@
 Text Label 6300 2150 0    50   ~ 0
 ADC_BATT
-Text Label 16100 6550 2    50   ~ 0
-OPENLOG_RX
-Text Label 16100 6450 2    50   ~ 0
-OPENLOG_TX
-Text Label 7500 5800 0    50   ~ 0
-OPENLOG_RX
-Text Label 7500 5700 0    50   ~ 0
-OPENLOG_TX
 Text Label 15700 5000 2    50   ~ 0
 GPS_RX
@@
 $EndComp
 $Comp
-L power:GND #PWR051
-U 1 1 610B2F7E
-P 15800 6050
-F 0 "#PWR051" H 15800 5800 50  0001 C CNN
-F 1 "GND" H 15805 5877 50  0000 C CNN
-F 2 "" H 15800 6050 50  0001 C CNN
-F 3 "" H 15800 6050 50  0001 C CNN
-	1    15800 6050
-	1    0    0    -1
-$EndComp
-$Comp
 L power:GND #PWR01
 U 1 1 610B7464
@@
 Wire Wire Line
 	15700 5100 15700 5350
-Wire Wire Line
-	16100 6250 15900 6250
-Wire Wire Line
-	15900 6250 15900 6050
-Wire Wire Line
-	15900 6050 15800 6050
-Wire Wire Line
-	15550 6300 15550 6350
-Wire Wire Line
-	15550 6350 16100 6350
 Wire Wire Line
 	13100 4850 13750 4850
@@
 Wire Wire Line
 	15250 5200 15950 5200
-$Comp
-L power:+3.3V #PWR049
-U 1 1 610A5207
-P 15550 6300
-F 0 "#PWR049" H 15550 6150 50  0001 C CNN
-F 1 "+3.3V" H 15565 6473 50  0000 C CNN
-F 2 "" H 15550 6300 50  0001 C CNN
-F 3 "" H 15550 6300 50  0001 C CNN
-	1    15550 6300
-	1    0    0    -1
-$EndComp
 Text Label 13750 4750 2    50   ~ 0
 NX_SDA
@@
 F 0 "U2" H 3250 5465 50  0000 C CNN
 F 1 "TDK_I3A4W008A033V" H 3250 5374 50  0000 C CNN
-F 2 "" H 2750 5300 50  0001 C CNN
+F 2 "ASTRA_Footprints:Power_Supply_32nd_Brick" H 2750 5300 50  0001 C CNN
 F 3 "" H 2750 5300 50  0001 C CNN
 F 4 "285-2720-ND" H 3250 5000 50  0001 C CNN "Digikey Part Num"
@@
 F 0 "U3" H 3700 7465 50  0000 C CNN
 F 1 "TDK_I3A4W008A033V" H 3700 7374 50  0000 C CNN
-F 2 "" H 3200 7300 50  0001 C CNN
+F 2 "ASTRA_Footprints:Power_Supply_32nd_Brick" H 3200 7300 50  0001 C CNN
 F 3 "" H 3200 7300 50  0001 C CNN
 F 4 "285-2720-ND" H 3700 7000 50  0001 C CNN "Digikey Part Num"

Commit message: 24v power supply swapped
Parts:
- added C3, C4: 100u, Capacitor_SMD:CP_Elec_10x10, symbol Device:CP_Small
- added D5, D6: D_Schottky_Small, Diode_SMD:D_SOD-323_HandSoldering, symbol Device:D_Schottky_Small
- added J6: Conn_01x02, Connector_JST:JST_XH_B2B-XH-A_1x02_P2.50mm_Vertical, symbol Connector_Generic:Conn_01x02
- added Q3: Q_NMOS_GSD, Package_TO_SOT_SMD:SOT-23, symbol Device:Q_NMOS_GSD
- added R10: 80.6k, Resistor_SMD:R_0603_1608Metric, symbol Device:R_Small
- added R11: 10k, Resistor_SMD:R_0603_1608Metric, symbol Device:R_Small
- added R3: 100k, Resistor_SMD:R_0603_1608Metric, symbol Device:R_Small
- added U4: PYBE30-Q24-S24, ASTRA_Footprints:PYBE30, symbol ASTRA_Library:PYBE30-Q24-S24
- renumbered C3 to C5, C4 to C6, D8 to D10, D9 to D11, D10 to D12, D5 to D7, D6 to D8, D7 to D9, J9 to J10, J10 to J11, J11 to J12, J12 to J13, J13 to J14, J6 to J7, J7 to J8, J8 to J9, Q3 to Q4, Q4 to Q5, Q5 to Q6, Q6 to Q7, Q7 to Q8, R9 to R12, R10 to R13, R11 to R14, R12 to R15, R13 to R16, R14 to R17, R15 to R18, R3 to R4, R4 to R5, R5 to R6, R6 to R7, R7 to R8, R8 to R9, U9 to U10, U10 to U11, U4 to U5, U5 to U6, U6 to U7, U7 to U8, U8 to U9
Connections:
- net +3V3: now also D5.1 (K)
- net +BATT: now also C3.1, U4.1 (Vin)
- net GND: now also C3.2, C4.2, D6.2 (A), J6.2 (Pin_2), Q3.2 (S), R11.2, R3.2, U4.2 (GND), U4.5 (0V)
- net 24V_Disable: now reaches U5.24 (P32)
- net 24V_Disable: now also Q3.1 (G), R3.1
- net ADC_24V: now reaches U5.44 (P22)
- net ADC_24V: now also D5.2 (A), D6.1 (K), R10.2, R11.1
- new net: Q3.3 (D), U4.3 (CTRL)
- new net +24V: C4.1, J6.1 (Pin_1), R10.1, U4.6 (+Vo)
Other:
- note added: "Comms Power Supply"
- note removed: "ANT connection off-board"
- note removed: "off-board PSD-30B-24"

Commit message: fixed a small error with footprints
Parts:
- U10, U8, U9: footprint Package_TO_SOT_SMD:SOT-23 -> Connector_JST:JST_PH_B3B-PH-K_1x03_P2.00mm_Vertical
- U6, U7: footprint Package_TO_SOT_SMD:SOT-23 -> Package_TO_SOT_THT:TO-92
Changed lines of the file:
@@
 F 0 "U6" H 8820 2046 50  0000 R CNN
 F 1 "Analog Temp Sensor" H 8820 1955 50  0000 R CNN
-F 2 "Package_TO_SOT_SMD:SOT-23" H 9150 1600 50  0001 C CNN
+F 2 "Package_TO_SOT_THT:TO-92" H 9150 1600 50  0001 C CNN
 F 3 "http://ww1.microchip.com/downloads/en/DeviceDoc/21942e.pdf" H 9000 2250 50  0001 C CNN
 F 4 "296-46127-1-ND" H 9150 2000 50  0001 C CNN "Digikey Part Num"
@@
 F 0 "U7" H 9720 2046 50  0000 R CNN
 F 1 "Analog Temp Sensor" H 9720 1955 50  0000 R CNN
-F 2 "Package_TO_SOT_SMD:SOT-23" H 10050 1600 50  0001 C CNN
+F 2 "Package_TO_SOT_THT:TO-92" H 10050 1600 50  0001 C CNN
 F 3 "http://ww1.microchip.com/downloads/en/DeviceDoc/21942e.pdf" H 9900 2250 50  0001 C CNN
 F 4 "296-46127-1-ND" H 10050 2000 50  0001 C CNN "Digikey Part Num"
@@
 F 0 "U8" H 10620 2046 50  0000 R CNN
 F 1 "Analog Temp Sensor" H 10620 1955 50  0000 R CNN
-F 2 "Package_TO_SOT_SMD:SOT-23" H 10950 1600 50  0001 C CNN
+F 2 "Connector_JST:JST_PH_B3B-PH-K_1x03_P2.00mm_Vertical" H 10950 1600 50  0001 C CNN
 F 3 "http://ww1.microchip.com/downloads/en/DeviceDoc/21942e.pdf" H 10800 2250 50  0001 C CNN
 F 4 "296-46127-1-ND" H 10950 2000 50  0001 C CNN "Digikey Part Num"
@@
 F 0 "U9" H 11520 2046 50  0000 R CNN
 F 1 "Analog Temp Sensor" H 11520 1955 50  0000 R CNN
-F 2 "Package_TO_SOT_SMD:SOT-23" H 11850 1600 50  0001 C CNN
+F 2 "Connector_JST:JST_PH_B3B-PH-K_1x03_P2.00mm_Vertical" H 11850 1600 50  0001 C CNN
 F 3 "http://ww1.microchip.com/downloads/en/DeviceDoc/21942e.pdf" H 11700 2250 50  0001 C CNN
 F 4 "296-46127-1-ND" H 11850 2000 50  0001 C CNN "Digikey Part Num"
@@
 F 0 "U10" H 12420 2046 50  0000 R CNN
 F 1 "Analog Temp Sensor" H 12420 1955 50  0000 R CNN
-F 2 "Package_TO_SOT_SMD:SOT-23" H 12750 1600 50  0001 C CNN
+F 2 "Connector_JST:JST_PH_B3B-PH-K_1x03_P2.00mm_Vertical" H 12750 1600 50  0001 C CNN
 F 3 "http://ww1.microchip.com/downloads/en/DeviceDoc/21942e.pdf" H 12600 2250 50  0001 C CNN
 F 4 "296-46127-1-ND" H 12750 2000 50  0001 C CNN "Digikey Part Num"

Commit message: Removed 24V connector, Changed net switch power bus, changed motor driver connector
Parts:
- removed C3, C4: 100u, Capacitor_SMD:CP_Elec_10x10, symbol Device:CP_Small
- removed J10, J11, J12, J13, J14, J9: FSESC_6.6_COMM, Connector_JST:JST_PH_B8B-PH-K_1x08_P2.00mm_Vertical, symbol ASTRA_Library:FSESC_6.6_COMM
- removed J6: Conn_01x02, Connector_JST:JST_XH_B2B-XH-A_1x02_P2.50mm_Vertical, symbol Connector_Generic:Conn_01x02
- removed Q3: Q_NMOS_GSD, Package_TO_SOT_SMD:SOT-23, symbol Device:Q_NMOS_GSD
- removed R3: 100k, Resistor_SMD:R_0603_1608Metric, symbol Device:R_Small
- removed U4: PYBE30-Q24-S24, ASTRA_Footprints:PYBE30, symbol ASTRA_Library:PYBE30-Q24-S24
- added J10, J11, J12, J13, J6, J9: FSESC_6.6_COMM_Minimal, Connector_JST:JST_PH_B3B-PH-K_1x03_P2.00mm_Vertical, symbol ASTRA_Library:FSESC_6.6_COMM_Minimal
Connections:
- net +12V: no longer J4.1 (Pin_1)
- net +5V: now also J4.1 (Pin_1)
- net ADC_24V: no longer U5.44 (P22)
- net GND: now also J10.1 (GND), J11.1 (GND), J12.1 (GND), J13.1 (GND), J6.1 (GND), J9.1 (GND)
- net M1_RX: now also J6.2 (RX)
- net M1_TX: now also J6.3 (TX)
- net M2_RX: now also J9.2 (RX)
- net M2_TX: now also J9.3 (TX)
- net M3_RX: now also J10.2 (RX)
- net M3_TX: now also J10.3 (TX)
- net M4_RX: now also J11.2 (RX)
- net M4_TX: now also J11.3 (TX)
- net M5_RX: now also J12.2 (RX)
- net M5_TX: now also J12.3 (TX)
- net M6_RX: now also J13.2 (RX)
- net M6_TX: now also J13.3 (TX)
- net 24V_Disable: no longer names the net of U5.24 (P32)
- no-connect marks 25 -> 6
Other:
- note removed: "24v"
- note removed: "Comms Power Supply"
