File: main-board/main-board.sch (KiCad schematic (older format))
At the start: 73 parts, among them J1 NVIDIA_Jetson_NX_Dev_40pin_Co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, J10 FSESC_6.6_COMM_Minimal, J11 FSESC_6.6_COMM_Minimal, J12 FSESC_6.6_COMM_Minimal, J13 FSESC_6.6_COMM_Minimal, J14 ArducamPTZ, J15 Angle Sensor, J2 NVIDIA_Jetson_NX_Dev_Button_C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, J3 Conn_01x02, J4 Conn_01x02, J5 Conn_01x02, J6 FSESC_6.6_COMM_Minimal, J7 QWIIC_Generic_Conn, J8 Conn_01x03, J9 FSESC_6.6_COMM_Minimal, M1 Fan_3pin, M2 Fan_3pin, M3 Fan_3pin, Q1 Q_NMOS_GSD, Q4 Q_NMOS_GSD, Q5 Q_NMOS_GSD, Q6 Q_NMOS_GSD, Q7 Q_NMOS_GSD, Q8 Q_NMOS_GSD, U1 RFM95W_Adafruit_Breakout, U10 Analog Temp Sensor, U11 Adafruit_GPS_V3, U12 SN74AHCT125D, U2 TDK_I3A4W008A033V, U3 TDK_I3A4W008A033V, U5 Teensy_4.1, U6 Analog Temp Sensor, U7 Analog Temp Sensor, U8 Analog Temp Sensor, U9 Analog Temp Sensor

Commit message: Indicator LEDs
Parts:
- added D13, D14, D5, D6: G, LED_SMD:LED_0603_1608Metric_Pad1.05x0.95mm_HandSolder, symbol Device:LED_Small
- added R10: 1k, Resistor_SMD:R_0603_1608Metric, symbol Device:R_Small
- added R11: 3.3k, Resistor_SMD:R_0603_1608Metric, symbol Device:R_Small
- added R2: 10, Resistor_SMD:R_0603_1608Metric, symbol Device:R_Small
- added R3: 180, Resistor_SMD:R_0603_1608Metric, symbol Device:R_Small
Connections:
- net +12V: now also D13.2 (A)
- net +3V3: now also D5.2 (A)
- net +5V: now also D6.2 (A)
- net +BATT: now also D14.2 (A)
- net GND: now also R10.2, R11.2, R2.2, R3.2
- new net: D5.1 (K), R2.1
- new net: D6.1 (K), R3.1
- new net: D13.1 (K), R10.1
- new net: D14.1 (K), R11.1
Changed lines of the file:
@@
+	1    0    0    -1
+$EndComp
+$Comp
+L Device:LED_Small D5
+U 1 1 623ACB6F
+P 2500 11600
+F 0 "D5" V 2546 11530 50  0000 R CNN
+F 1 "G" V 2455 11530 50  0000 R CNN
+F 2 "LED_SMD:LED_0603_1608Metric_Pad1.05x0.95mm_HandSolder" V 2500 11600 50  0001 C CNN
+F 3 "~" V 2500 11600 50  0001 C CNN
+F 4 "732-4971-1-ND" V 2500 11600 50  0001 C CNN "Digikey Part Num"
+	1    2500 11600
+	0    -1   -1   0
+$EndComp
+$Comp
+L power:+3.3V #PWR05
+U 1 1 623B0140
+P 2500 11350
+F 0 "#PWR05" H 2500 11200 50  0001 C CNN
+F 1 "+3.3V" H 2515 11523 50  0000 C CNN
+F 2 "" H 2500 11350 50  0001 C CNN
+F 3 "" H 2500 11350 50  0001 C CNN
+	1    2500 11350
+	1    0    0    -1
+$EndComp
+$Comp
+L power:+5V #PWR013
+U 1 1 623B2688
+P 2850 11350
+F 0 "#PWR013" H 2850 11200 50  0001 C CNN
+F 1 "+5V" H 2865 11523 50  0000 C CNN
+F 2 "" H 2850 11350 50  0001 C CNN
+F 3 "" H 2850 11350 50  0001 C CNN
+	1    2850 11350
+	1    0    0    -1
+$EndComp
+$Comp
+L power:+12V #PWR019
+U 1 1 623B3A32
+P 3200 11350
+F 0 "#PWR019" H 3200 11200 50  0001 C CNN
+F 1 "+12V" H 3215 11523 50  0000 C CNN
+F 2 "" H 3200 11350 50  0001 C CNN
+F 3 "" H 3200 11350 50  0001 C CNN
+	1    3200 11350
+	1    0    0    -1
+$EndComp
+$Comp
+L power:+BATT #PWR023
+U 1 1 623B50E5
+P 3550 11350
+F 0 "#PWR023" H 3550 11200 50  0001 C CNN
+F 1 "+BATT" H 3565 11523 50  0000 C CNN
+F 2 "" H 3550 11350 50  0001 C CNN
+F 3 "" H 3550 11350 50  0001 C CNN
+	1    3550 11350
+	1    0    0    -1
+$EndComp
+$Comp
+L Device:R_Small R2
+U 1 1 623B760B
+P 2500 11900
+F 0 "R2" H 2559 11946 50  0000 L CNN
+F 1 "10" H 2559 11855 50  0000 L CNN
+F 2 "Resistor_SMD:R_0603_1608Metric" H 2500 11900 50  0001 C CNN
+F 3 "~" H 2500 11900 50  0001 C CNN
+F 4 "311-10.0HRCT-ND" H 2500 11900 50  0001 C CNN "Digikey Part Num"
+	1    2500 11900
+	1    0    0    -1
+$EndComp
+$Comp
+L power:GND #PWR010
+U 1 1 623B86FD
+P 2500 12100
+F 0 "#PWR010" H 2500 11850 50  0001 C CNN
+F 1 "GND" H 2505 11927 50  0000 C CNN
+F 2 "" H 2500 12100 50  0001 C CNN
+F 3 "" H 2500 12100 50  0001 C CNN
+	1    2500 12100
+	1    0    0    -1
+$EndComp
+Wire Wire Line
+	2500 12100 2500 12000
+Wire Wire Line
+	2500 11800 2500 11700
+Wire Wire Line
+	2500 11500 2500 11350
+$Comp
+L Device:LED_Small D6
+U 1 1 623F4A14
+P 2850 11600
+F 0 "D6" V 2896 11530 50  0000 R CNN
+F 1 "G" V 2805 11530 50  0000 R CNN
+F 2 "LED_SMD:LED_0603_1608Metric_Pad1.05x0.95mm_HandSolder" V 2850 11600 50  0001 C CNN
+F 3 "~" V 2850 11600 50  0001 C CNN
+F 4 "732-4971-1-ND" V 2850 11600 50  0001 C CNN "Digikey Part Num"
+	1    2850 11600
+	0    -1   -1   0
+$EndComp
+$Comp
+L power:GND #PWR014
+U 1 1 623F4A21
+P 2850 12100
+F 0 "#PWR014" H 2850 11850 50  0001 C CNN
+F 1 "GND" H 2855 11927 50  0000 C CNN
+F 2 "" H 2850 12100 50  0001 C CNN
+F 3 "" H 2850 12100 50  0001 C CNN
+	1    2850 12100
+	1    0    0    -1
+$EndComp
+Wire Wire Line
+	2850 12100 2850 12000
+Wire Wire Line
+	2850 11800 2850 11700
+Wire Wire Line
+	2850 11500 2850 11350
+$Comp
+L Device:LED_Small D13
+U 1 1 6240758A
+P 3200 11600
+F 0 "D13" V 3246 11530 50  0000 R CNN
+F 1 "G" V 3155 11530 50  0000 R CNN
+F 2 "LED_SMD:LED_0603_1608Metric_Pad1.05x0.95mm_HandSolder" V 3200 11600 50  0001 C CNN
+F 3 "~" V 3200 11600 50  0001 C CNN
+F 4 "732-4971-1-ND" V 3200 11600 50  0001 C CNN "Digikey Part Num"
+	1    3200 11600
+	0    -1   -1   0
+$EndComp
+$Comp
+L power:GND #PWR022
+U 1 1 62407597
+P 3200 12100
+F 0 "#PWR022" H 3200 11850 50  0001 C CNN
+F 1 "GND" H 3205 11927 50  0000 C CNN
+F 2 "" H 3200 12100 50  0001 C CNN
+F 3 "" H 3200 12100 50  0001 C CNN
+	1    3200 12100
+	1    0    0    -1
+$EndComp
+Wire Wire Line
+	3200 12100 3200 12000
+Wire Wire Line
+	3200 11800 3200 11700
+Wire Wire Line
+	3200 11500 3200 11350
+$Comp
+L Device:LED_Small D14
+U 1 1 6241A756
+P 3550 11600
+F 0 "D14" V 3596 11530 50  0000 R CNN
+F 1 "G" V 3505 11530 50  0000 R CNN
+F 2 "LED_SMD:LED_0603_1608Metric_Pad1.05x0.95mm_HandSolder" V 3550 11600 50  0001 C CNN
+F 3 "~" V 3550 11600 50  0001 C CNN
+F 4 "732-4971-1-ND" V 3550 11600 50  0001 C CNN "Digikey Part Num"
+	1    3550 11600
+	0    -1   -1   0
+$EndComp
+$Comp
+L power:GND #PWR033
+U 1 1 6241A763
+P 3550 12100
+F 0 "#PWR033" H 3550 11850 50  0001 C CNN
+F 1 "GND" H 3555 11927 50  0000 C CNN
+F 2 "" H 3550 12100 50  0001 C CNN
+F 3 "" H 3550 12100 50  0001 C CNN
+	1    3550 12100
+	1    0    0    -1
+$EndComp
+Wire Wire Line
+	3550 12100 3550 12000
+Wire Wire Line
+	3550 11800 3550 11700
+Wire Wire Line
+	3550 11500 3550 11350
+$Comp
+L Device:R_Small R10
+U 1 1 62407591
+P 3200 11900
+F 0 "R10" H 3259 11946 50  0000 L CNN
+F 1 "1k" H 3259 11855 50  0000 L CNN
+F 2 "Resistor_SMD:R_0603_1608Metric" H 3200 11900 50  0001 C CNN
+F 3 "~" H 3200 11900 50  0001 C CNN
+F 4 "311-1.00KHRCT-ND" H 3200 11900 50  0001 C CNN "Digikey Part Num"
+	1    3200 11900
+	1    0    0    -1
+$EndComp
+$Comp
+L Device:R_Small R11
+U 1 1 6241A75D
+P 3550 11900
+F 0 "R11" H 3609 11946 50  0000 L CNN
+F 1 "3.3k" H 3609 11855 50  0000 L CNN
+F 2 "Resistor_SMD:R_0603_1608Metric" H 3550 11900 50  0001 C CNN
+F 3 "~" H 3550 11900 50  0001 C CNN
+F 4 "311-3.30KHRCT-ND" H 3550 11900 50  0001 C CNN "Digikey Part Num"
+	1    3550 11900
+	1    0    0    -1
+$EndComp
+$Comp
+L Device:R_Small R3
+U 1 1 623F4A1B
+P 2850 11900
+F 0 "R3" H 2909 11946 50  0000 L CNN
+F 1 "180" H 2909 11855 50  0000 L CNN
+F 2 "Resistor_SMD:R_0603_1608Metric" H 2850 11900 50  0001 C CNN
+F 3 "~" H 2850 11900 50  0001 C CNN
+F 4 "311-180HRCT-ND" H 2850 11900 50  0001 C CNN "Digikey Part Num"
+	1    2850 11900
 	1    0    0    -1
 $EndComp
